Commit message: Añadidas colisiones e inercias. Solo funciona en Gazebo si quito los stl.

File: src/articubot_one/description/robot.urdf.xacro (robot description, xacro)
@@ -1,4 +1,4 @@
 <?xml version="1.0"?>
 <robot xmlns:xacro="http://www.ros.org/wiki/xacro"  name="robot">
-    <xacro:include filename="robot_core.xacro" />
+    <xacro:include filename="robot_base.xacro" />
 </robot>

File: src/articubot_one/description/robot_base.xacro (robot description, xacro)
@@ -1,4 +1,4 @@
 <?xml version="1.0"?>
-<robot xmlns:xacro="http://ros.org/wiki/xacro" name="robot_base" >
+<robot xmlns:xacro="http://ros.org/wiki/xacro">
     <xacro:include filename="robot_essentials.xacro"/>
     <link name="base_link">
@@ -6,5 +6,6 @@
             <origin xyz="0 0 0" rpy="1.5707963267949 0 3.14"/>
             <geometry>
-                <mesh filename="package://articubot_one/meshes/robot_base.stl"/>
+                <!-- <mesh filename="package://articubot_one/meshes/robot_base.stl"/> -->
+                <box size="0.65 0.2 0.4"/>
             </geometry>
             <material name="">
@@ -12,4 +13,13 @@
             </material>
         </visual>
+        <collision>
+            <origin xyz="0 0 0.05" rpy="1.5707963267949 0 3.14"/>
+            <geometry>
+                <box size="0.650 0.200 0.400"/>
+            </geometry>
+        </collision>
+        <xacro:inertial_box mass="47" x="0.650" y="0.200" z="0.400">
+            <origin xyz="0 0 0.05" rpy="0 0 0"/>
+        </xacro:inertial_box>
     </link>
     <!-- Ruedas -->
@@ -27,9 +37,8 @@
     <link name="front_left_wheel">
         <visual>
-            <origin
-            xyz="0 0 0"
-            rpy="0 0 0" />
+            <origin xyz="0 0 0" rpy="0 0 0" />
             <geometry>
-                <mesh filename="package://articubot_one/meshes/wheel.stl" />
+                <!-- <mesh filename="package://articubot_one/meshes/wheel.stl" /> -->
+                <cylinder radius="0.1" length="0.05"/>
             </geometry>
             <material name="">
@@ -37,4 +46,13 @@
             </material>
         </visual>
+        <collision>
+            <origin xyz="0 0 0" rpy="0 0 0" />
+            <geometry>
+                <cylinder radius="0.1" length="0.1"/>
+            </geometry>
+        </collision>
+        <xacro:inertial_cylinder mass="2" length="0.1" radius="0.1">
+            <origin xyz="0 0 0" rpy="0 0 0"/>
+        </xacro:inertial_cylinder>
     </link>
     <joint name="front_left_wheel_joint" type="continuous">
@@ -43,5 +61,5 @@
         <child link ="front_left_wheel"/>
         <origin rpy ="${-pi/2} 0 0" xyz= "0.220 0.250 0"/>
-  </joint>
+    </joint>
   <!-- Front right wheel -->
     <link name="front_right_wheel">
@@ -51,5 +69,6 @@
             rpy="0 0 0" />
             <geometry>
-                <mesh filename="package://articubot_one/meshes/wheel.stl" />
+                <!-- <mesh filename="package://articubot_one/meshes/wheel.stl" /> -->
+                <cylinder radius="0.1" length="0.05"/>
             </geometry>
             <material name="">
@@ -57,4 +76,13 @@
             </material>
         </visual>
+        <collision>
+            <origin xyz="0 0 0" rpy="0 0 0" />
+            <geometry>
+                <cylinder radius="0.1" length="0.1"/>
+            </geometry>
+        </collision>
+        <xacro:inertial_cylinder mass="2" length="0.1" radius="0.1">
+            <origin xyz="0 0 0" rpy="0 0 0"/>
+        </xacro:inertial_cylinder>
     </link>
     <joint name="front_right_wheel_joint" type="continuous">
@@ -63,5 +91,5 @@
         <child link ="front_right_wheel"/>
         <origin rpy ="${pi/2} 0 0" xyz= "0.220 -0.250 0"/>
-  </joint>
+    </joint>
   <!-- Rear left wheel -->
     <link name="rear_left_wheel">
@@ -71,5 +99,6 @@
             rpy="0 0 0" />
             <geometry>
-                <mesh filename="package://articubot_one/meshes/wheel.stl" />
+                <!-- <mesh filename="package://articubot_one/meshes/wheel.stl" /> -->
+                <cylinder radius="0.1" length="0.05"/>
             </geometry>
             <material name="">
@@ -77,4 +106,13 @@
             </material>
         </visual>
+        <collision>
+            <origin xyz="0 0 0" rpy="0 0 0" />
+            <geometry>
+                <cylinder radius="0.1" length="0.1"/>
+            </geometry>
+        </collision>
+        <xacro:inertial_cylinder mass="2" length="0.1" radius="0.1">
+            <origin xyz="0 0 0" rpy="0 0 0"/>
+        </xacro:inertial_cylinder>
     </link>
     <joint name="rear_left_wheel_joint" type="continuous">
@@ -91,5 +129,6 @@
             rpy="0 0 0" />
             <geometry>
-                <mesh filename="package://articubot_one/meshes/wheel.stl" />
+                <!-- <mesh filename="package://articubot_one/meshes/wheel.stl" /> -->
+                <cylinder radius="0.1" length="0.05"/>
             </geometry>
             <material name="">
@@ -97,4 +136,13 @@
             </material>
         </visual>
+        <collision>
+            <origin xyz="0 0 0" rpy="0 0 0" />
+            <geometry>
+                <cylinder radius="0.1" length="0.1"/>
+            </geometry>
+        </collision>
+        <xacro:inertial_cylinder mass="2" length="0.1" radius="0.1">
+            <origin xyz="0 0 0" rpy="0 0 0"/>
+        </xacro:inertial_cylinder>
     </link>
     <joint name="rear_right_wheel_joint" type="continuous">
@@ -103,4 +151,4 @@
         <child link ="rear_right_wheel"/>
         <origin rpy ="${pi/2} 0 0" xyz= "-0.220 -0.250 0"/>
-  </joint>
+    </joint>
 </robot>

File: src/articubot_one/description/robot_essentials.xacro (robot description, xacro)
@@ -1,4 +1,4 @@
 <?xml version="1.0"?>
-<robot xmlns:xacro="http://www.ros.org/wiki/xacro" name="robot_essentials">
+<robot xmlns:xacro="http://www.ros.org/wiki/xacro">
 <!-- Macro para las ruedas -->
 <xacro:macro name="robot_wheel" params="prefix">
@@ -26,3 +26,22 @@
   </joint>
 </xacro:macro>
+<!-- Macros para las INERCIAS -->
+<xacro:macro name="inertial_box" params="mass x y z *origin">
+    <inertial>
+        <xacro:insert_block name="origin"/>
+        <mass value="${mass}" />
+        <inertia ixx="${(1/12) * mass * (y*y+z*z)}" ixy="0.0" ixz="0.0"
+                iyy="${(1/12) * mass * (x*x+z*z)}" iyz="0.0"
+                izz="${(1/12) * mass * (x*x+y*y)}" />
+    </inertial>
+</xacro:macro>
+<xacro:macro name="inertial_cylinder" params="mass length radius *origin">
+    <inertial>
+        <xacro:insert_block name="origin"/>
+        <mass value="${mass}" />
+        <inertia ixx="${(1/12) * mass * (3*radius*radius + length*length)}" ixy="0.0" ixz="0.0"
+                iyy="${(1/12) * mass * (3*radius*radius + length*length)}" iyz="0.0"
+                izz="${(1/2) * mass * (radius*radius)}" />
+    </inertial>
+</xacro:macro>
 </robot>
