Commit message: Primer uso de Navigation2

File: install/bulldog_description/share/bulldog_description/urdf/bulldog/bulldog.urdf.xacro (robot description, xacro)
@@ -28,9 +28,4 @@
       </geometry>
     </collision>
-  </link>
-  <gazebo reference="base_link">
-    <material>Gazebo/FlatBlack</material>
-  </gazebo>
-  <link name="inertial_link">
     <inertial>
       <mass value="40" />
@@ -38,7 +33,14 @@
       <inertia ixx="0.7" ixy="-0.03" ixz="-0.15" iyy="2" iyz="-0.01" izz="4" />
     </inertial>
-    <!-- <xacro:inertial_box mass="40" x="${base_x_size}" y="${base_y_size}" z="${base_z_size}">
-        <origin xyz="0 0 0.1" rpy="0 0 0"/>
-    </xacro:inertial_box> -->
+  </link>
+  <gazebo reference="base_link">
+    <material>Gazebo/FlatBlack</material>
+  </gazebo>
+  <!-- <link name="inertial_link">
+    <inertial>
+      <mass value="40" />
+      <origin xyz="0 0 0.1" />
+      <inertia ixx="0.7" ixy="-0.03" ixz="-0.15" iyy="2" iyz="-0.01" izz="4" />
+    </inertial>
   </link>
   <joint name="inertial_joint" type="fixed">
@@ -46,5 +48,5 @@
     <parent link="base_link" />
     <child link="inertial_link" />
-  </joint>
+  </joint> -->
   <link name="top_plate_link">
     <visual>
@@ -64,5 +66,5 @@
     <child link="top_plate_link" />
   </joint>
-  <link name="imu_link"/>
+  <!-- <link name="imu_link"/>
   <joint name="imu_joint" type="fixed">
     <origin xyz="0 0 0" rpy="0 0 0" />
@@ -70,6 +72,6 @@
     <child link="imu_link" />
   </joint>
-  <gazebo reference="imu_link" />
-  <link name="rslidar"/>
+  <gazebo reference="imu_link" /> -->
+  <!-- <link name="rslidar"/>
   <joint name="rslidar_joint" type="fixed">
     <origin xyz="-0.045 0 0.6" rpy="0 0 0" />
@@ -77,5 +79,5 @@
     <child link="rslidar" />
   </joint>
-  <gazebo reference="rslidar" />
+  <gazebo reference="rslidar" /> -->
   <xacro:bulldog_wheel wheel_prefix="front_left">
     <origin xyz="0.27937 0.285 0.0435" rpy="0 0 0" />

File: install/mobile_manipulator/share/mobile_manipulator/urdf/mm.urdf.xacro (robot description, xacro)
@@ -1,5 +1,5 @@
 <?xml version="1.0"?>
 <robot name="mobile_manipulator" xmlns:xacro="http://ros.org/wiki/xacro">
-    <xacro:arg name="laser_enabled" default="false" />
+    <!-- <xacro:arg name="laser_enabled" default="false" /> -->
     <xacro:arg name="arm_enabled" default="true" />
     <xacro:include filename="$(find bulldog_description)/urdf/bulldog/bulldog.urdf.xacro" />
@@ -15,12 +15,78 @@
         </joint>
     </xacro:if>
-    <xacro:if value="$(arg laser_enabled)">
+    <!-- <xacro:if value="$(arg laser_enabled)">
         <xacro:laser_plate />
-        <!-- <sick_lms1xx frame="laser_link" topic="scan"/> -->
-        <!-- <joint name="laser_mount_joint" type="fixed">
+        <sick_lms1xx frame="laser_link" topic="scan"/>
+        <joint name="laser_mount_joint" type="fixed">
         <origin xyz="0.015 0 0.044" rpy="${M_PI} 0 0" />
         <parent link="laser_plate_link" />
         <child link="laser_link" />
-        </joint> -->
-    </xacro:if>
+        </joint>
+    </xacro:if> -->
+    <!-- LASER -->
+    <link name="laser_link">
+        <collision>
+            <origin xyz="0 0 0" rpy="0 0 0"/>
+            <geometry>
+                <box size="0.1 0.1 0.1"/>
+            </geometry>
+        </collision>
+        <visual>
+            <origin xyz="0 0 0" rpy="0 0 0"/>
+            <geometry>
+                <box size="0.05 0.05 0.05"/>
+            </geometry>
+        </visual>
+        <inertial>
+            <mass value="1e-5" />
+            <origin xyz="0 0 0" rpy="0 0 0"/>
+            <inertia ixx="1e-6" ixy="0" ixz="0" iyy="1e-6" iyz="0" izz="1e-6" />
+        </inertial>
+    </link>
+    <joint name="laser_joint" type="fixed">
+        <axis xyz="0 1 0" />
+        <origin xyz="0.430 0 0.20" rpy="0 0 0"/>
+        <parent link="base_link"/>
+        <child link="laser_link"/>
+    </joint>
+    <gazebo reference="laser_link">
+        <sensor type="ray" name="laser">
+            <pose>0 0 0 0 0 0</pose>
+            <visualize>true</visualize>
+            <update_rate>10</update_rate>
+            <ray>
+                <scan>
+                    <horizontal>
+                        <samples>720</samples>
+                        <resolution>1</resolution>
+                        <min_angle>-1.570796</min_angle>
+                        <max_angle>1.570796</max_angle>
+                    </horizontal>
+                </scan>
+                <range>
+                    <min>0.30</min>
+                    <max>12.0</max>
+                    <!-- <resolution>0.01</resolution> -->
+                </range>
+            </ray>
+            <!-- <plugin name="gazebo_ros_head_hokuyo_controller" filename="libgazebo_ros_laser.so">
+                <topicName>/scan</topicName>
+                <frameName>laser_link</frameName>
+            </plugin> -->
+            <plugin name="laser_controller" filename="libgazebo_ros_ray_sensor.so">
+                <ros>
+                    <argument>~/out:=scan</argument>
+                </ros>
+                <output_type>sensor_msgs/LaserScan</output_type>
+                <frame_name>laser_link</frame_name>
+            </plugin>
+        </sensor>
+    </gazebo>
+    <!-- BASE FOOTPRINT-->
+    <joint name="base_footprint_joint" type="fixed">
+        <parent link="base_link" />
+        <child link="base_footprint" />
+        <origin xyz="0 0 0" rpy="0 0 0" />
+    </joint>
+    <link name="base_footprint"/>
 </robot>

Commit message: Reach Goal node creado aunque no funcionan correctamente las transformaciones

File: install/bulldog_description/share/bulldog_description/urdf/bulldog/bulldog.urdf.xacro (robot description, xacro)
@@ -29,5 +29,6 @@
     </collision>
     <inertial>
-      <mass value="40" />
+      <!-- <mass value="40" /> -->
+      <mass value="100" />
       <origin xyz="0 0 0.1" />
       <inertia ixx="0.7" ixy="-0.03" ixz="-0.15" iyy="2" iyz="-0.01" izz="4" />

File: src/ur5_ros2_gazebo/urdf/ur5.urdf.xacro (robot description, xacro)
@@ -87,7 +87,7 @@
   <!-- CELL LAYOUT N1) UR5 ROBOT alone: -->
   <xacro:if value="${cell_layout_1}">
-    <joint name="world-base_link-fixed" type="fixed">
+    <joint name="world-base_0-fixed" type="fixed">
       <parent link="world"/>
-      <child link="base_link"/>
+      <child link="base_0"/>
     </joint>
   </xacro:if>
@@ -126,5 +126,5 @@
     <joint name="ur_joint" type="fixed">
       <parent link="ur_base" />
-      <child link = "base_link" />
+      <child link = "base_0" />
       <origin xyz="0.0 0.0 0.655" rpy="0.0 0.0 0.0" />
     </joint>

File: src/ur5_ros2_gazebo/urdf/ur5_macro.urdf.xacro (robot description, xacro)
@@ -73,6 +73,6 @@
     <!-- ***** ur5 ROBOT .urdf SERIAL CHAIN *****-->
     <!-- Links: -->
-    <link name="${prefix}base_link"/>
-    <link name="${prefix}base_link_inertia">
+    <link name="${prefix}base_0"/>
+    <link name="${prefix}base_0_inertia">
       <visual>
         <origin xyz="0 0 0" rpy="0 0 ${pi}"/>
@@ -215,7 +215,7 @@
     </link>
     <!-- Joints: -->
-    <joint name="${prefix}base_link-base_link_inertia" type="fixed">
-      <parent link="${prefix}base_link" />
-      <child link="${prefix}base_link_inertia" />
+    <joint name="${prefix}base_0-base_0_inertia" type="fixed">
+      <parent link="${prefix}base_0" />
+      <child link="${prefix}base_0_inertia" />
       <!-- 'base_link' is REP-103 aligned (so X+ forward), while the internal
            frames of the robot/controller have X+ pointing backwards.
@@ -226,5 +226,5 @@
     </joint>
     <joint name="${prefix}shoulder_pan_joint" type="revolute">
-      <parent link="${prefix}base_link_inertia" />
+      <parent link="${prefix}base_0_inertia" />
       <child link="${prefix}shoulder_link" />
       <origin xyz="${shoulder_x} ${shoulder_y} ${shoulder_z}" rpy="${shoulder_roll} ${shoulder_pitch} ${shoulder_yaw}" />
@@ -299,5 +299,5 @@
     <!-- ROS-Industrial 'base' frame - base_link to UR 'Base' Coordinates transform -->
     <link name="${prefix}base"/>
-    <joint name="${prefix}base_link-base_fixed_joint" type="fixed">
+    <joint name="${prefix}base_0-base_fixed_joint" type="fixed">
       <!-- Note the rotation over Z of pi radians - as base_link is REP-103
            aligned (i.e., has X+ forward, Y+ left and Z+ up), this is needed
@@ -306,5 +306,5 @@
       -->
       <origin xyz="0 0 0" rpy="0 0 ${pi}"/>
-      <parent link="${prefix}base_link"/>
+      <parent link="${prefix}base_0"/>
       <child link="${prefix}base"/>
     </joint>
