Commit message: Añadidos varios nodos para el movimiento del robot

File: install/bulldog_description/share/bulldog_description/urdf/bulldog/wheel.urdf.xacro (robot description, xacro)
@@ -31,5 +31,5 @@
     <mu1 value="1.0"/>
     <mu2 value="0.2"/>
-    <!-- <mu2 value="0.25"/> -->
+    <!-- <mu2 value="0.25"/> KEMPES engineers year-book 1985 (90th edition) -->
     <kp value="10000000.0" />
     <kd value="1.0" />

File: install/doosan_description/share/doosan_description/description/xacro/a0912.urdf.xacro (robot description, xacro)
@@ -1,25 +1,33 @@
 <?xml version="1.0"?>
 <robot xmlns:xacro="http://www.ros.org/wiki/xacro" name="a0912" >
-  <xacro:arg name="color"   default="blue"/>
-  <xacro:arg name="gripper" default="none"/>
-  <xacro:arg name="namespace" default=""/>
-  <xacro:property name="cr" value="$(arg color)"/>
-  <xacro:property name="gr" value="$(arg gripper)"/>
-  <xacro:if value="${cr == 'white'}">
-     <xacro:include filename="$(find doosan_description)/description/xacro/macro.a0912.white.xacro" />
-  </xacro:if>
-  <xacro:if value="${cr == 'blue'}">
-     <xacro:include filename="$(find doosan_description)/description/xacro/macro.a0912.blue.xacro" />
-  </xacro:if>
-  <xacro:if value="${gr == 'robotiq_2f'}">
-     <xacro:include filename="$(find doosan_description)/description/xacro/robotiq_2f.urdf.xacro" />
-  </xacro:if>
-  <xacro:a0912 namespace="$(arg namespace)"/>
-  <!-- World fixed joint-->
-  <!-- <link name="world" />
-  <joint name="world_fixed" type="fixed">
-    <origin xyz="0 0 0" rpy="0 0 0"/>
-    <parent link="world"/>
-    <child link="base_0"/>
-  </joint> -->
+   <xacro:arg name="color"   default="blue"/>
+   <xacro:arg name="gripper" default="none"/>
+   <xacro:arg name="namespace" default=""/>
+   <xacro:property name="cr" value="$(arg color)"/>
+   <xacro:property name="gr" value="$(arg gripper)"/>
+   <xacro:if value="${cr == 'white'}">
+      <xacro:include filename="$(find doosan_description)/description/xacro/macro.a0912.white.xacro" />
+   </xacro:if>
+   <xacro:if value="${cr == 'blue'}">
+      <xacro:include filename="$(find doosan_description)/description/xacro/macro.a0912.blue.xacro" />
+   </xacro:if>
+   <xacro:if value="${gr == 'robotiq_2f'}">
+      <xacro:include filename="$(find doosan_description)/description/xacro/robotiq_2f.urdf.xacro" />
+   </xacro:if>
+   <xacro:a0912 namespace="$(arg namespace)"/>
+   <!-- World fixed joint-->
+   <!-- <link name="world" />
+   <joint name="world_fixed" type="fixed">
+      <origin xyz="0 0 0" rpy="0 0 0"/>
+      <parent link="world"/>
+      <child link="base_0"/>
+   </joint> -->
+   <!-- GRIPPER -->
+   <xacro:include filename="$(find doosan_description)/description/xacro/gripper.xacro" />
+   <joint name="gripper_fixed" type="fixed">
+      <origin xyz="0 0.02 0.04" rpy="0 0 0"/>
+      <!-- origin xyz="0 0 0.5" rpy="0 0 0"/ -->
+      <parent link="link6"/>
+      <child link="gripper_link_base"/>
+   </joint>
 </robot>

File: install/doosan_description/share/doosan_description/description/xacro/macro.gazebo_config_control.xacro (robot description, xacro)
@@ -62,4 +62,23 @@
 	    		<state_interface name="effort"/>
 	    	</joint>
+			<!-- Prismatic joint for the gripper -->
+			<joint name="gripper_joint_left_1">
+				<command_interface name="position">
+					<param name="min">-0.04</param>
+					<param name="max">0.06</param>
+				</command_interface>
+				<state_interface name="position"/>
+				<state_interface name="velocity"/>
+				<state_interface name="effort"/>
+			</joint>
+			<joint name="gripper_joint_right_1">
+				<command_interface name="position">
+					<param name="min">0.04</param>
+					<param name="max">-0.06</param>
+				</command_interface>
+				<state_interface name="position"/>
+				<state_interface name="velocity"/>
+				<state_interface name="effort"/>
+			</joint>
 	  	</ros2_control>
 		<gazebo>

File: install/doosan_description/share/doosan_description/description/xacro/macro.internal_config.xacro (robot description, xacro)
@@ -69,4 +69,21 @@
       <minDepth>0.001</minDepth>
     </gazebo>
+    <!-- Gripper -->
+    <gazebo reference="gripper_link_left_1">
+      <kp>1000000.0</kp>
+      <kd>100.0</kd>
+      <mu1>30.0</mu1>
+      <mu2>30.0</mu2>
+      <maxVel>1.0</maxVel>
+      <minDepth>0.001</minDepth>
+    </gazebo>
+    <gazebo reference="gripper_link_right_1">
+      <kp>1000000.0</kp>
+      <kd>100.0</kd>
+      <mu1>30.0</mu1>
+      <mu2>30.0</mu2>
+      <maxVel>1.0</maxVel>
+      <minDepth>0.001</minDepth>
+    </gazebo>
 	</xacro:macro>
 </robot>

File: install/doosan_description/share/doosan_description/description/xacro/macro.transmission.xacro (robot description, xacro)
@@ -68,4 +68,25 @@
 			</actuator>
 		</transmission>
+		<!-- Gripper Transmission -->
+		<transmission name="gripper_tran_left_1">
+			<type>transmission_interface/SimpleTransmission</type>
+			<joint name="gripper_joint_left_1">
+				<hardwareInterface>hardware_interface/PositionJointInterface</hardwareInterface>
+			</joint>
+			<actuator name="gripper_motor_left_1">
+				<hardwareInterface>hardware_interface/PositionJointInterface</hardwareInterface>
+				<mechanicalReduction>1</mechanicalReduction>
+			</actuator>
+		</transmission>
+		<transmission name="gripper_tran_right_1">
+			<type>transmission_interface/SimpleTransmission</type>
+			<joint name="gripper_joint_right_1">
+				<hardwareInterface>hardware_interface/PositionJointInterface</hardwareInterface>
+			</joint>
+			<actuator name="gripper_motor_right_1">
+				<hardwareInterface>hardware_interface/PositionJointInterface</hardwareInterface>
+				<mechanicalReduction>1</mechanicalReduction>
+			</actuator>
+		</transmission>
 	</xacro:macro>
 </robot>

File: src/bulldog_description/urdf/bulldog/wheel.urdf.xacro (robot description, xacro)
@@ -2,6 +2,6 @@
 <robot name="bulldog_wheel" xmlns:xacro="http://ros.org/wiki/xacro">
   <!-- <xacro:include filename="$(find bulldog_description)/urdf/bulldog/inertial_macros.xacro" /> -->
-  <!-- <xacro:property name="wheel_length" value="0.142" />
-  <xacro:property name="wheel_radius" value="0.183" /> -->
+  <xacro:property name="wheel_length" value="0.142" />
+  <xacro:property name="wheel_radius" value="0.183" />
   <xacro:macro name="bulldog_wheel" params="wheel_prefix *joint_pose">
   <link name="${wheel_prefix}_wheel_link">
